File: plimsoll.kicad_sch (KiCad schematic)
At the start: 0 parts

Commit message: r0
Parts:
- added C1: 100n, Capacitor_SMD:C_0603_1608Metric, symbol Device:C_Small
- added C10, C6: 1u, Capacitor_SMD:C_0805_2012Metric, symbol Device:C
- added C11, C2, C4: 10u, Capacitor_SMD:C_0805_2012Metric, symbol Device:C
- added C12, C13, C14, C15, C16, C17, C3, C5, C7, C8, C9: 100n, Capacitor_SMD:C_0603_1608Metric, symbol Device:C
- added D1, D2: GRN, LED_SMD:LED_0805_2012Metric, symbol Device:LED
- added H1, H2: MountingHole, MountingHole:MountingHole_2.2mm_M2_ISO7380, symbol Mechanical:MountingHole
- added J1: TAG CONNECT, Connector:Tag-Connect_TC2030-IDC-NL_2x03_P1.27mm_Vertical, symbol Connector_Generic:Conn_01x06
- added J2: USB_C, Connector_USB:USB_C_Receptacle_G-Switch_GT-USB-7010ASV, symbol Connector:USB_C_Receptacle_USB2.0_16P
- added J3: Loadd Cell, Connector_JST:JST_XH_B4B-XH-A_1x04_P2.50mm_Vertical, symbol Connector_Generic:Conn_01x04
- added J4: Test Points, Connector_PinHeader_2.54mm:PinHeader_1x02_P2.54mm_Vertical, symbol Connector_Generic:Conn_01x02
- added JP1: S0, Jumper:SolderJumper-3_P1.3mm_Bridged12_RoundedPad1.0x1.5mm_NumberLabels, symbol Jumper:SolderJumper_3_Bridged12
- added JP2: S1, Jumper:SolderJumper-3_P1.3mm_Bridged12_RoundedPad1.0x1.5mm_NumberLabels, symbol Jumper:SolderJumper_3_Bridged12
- added R1: 1M, Resistor_SMD:R_0805_2012Metric, symbol Device:R
- added R10, R11, R12, R4: 10k, Resistor_SMD:R_0603_1608Metric, symbol Device:R_Small
- added R13, R14: 510, Resistor_SMD:R_0603_1608Metric, symbol Device:R_Small
- added R5, R6: 5k1, Resistor_SMD:R_0603_1608Metric, symbol Device:R_Small
- added R7, R8: 100, Resistor_SMD:R_0603_1608Metric, symbol Device:R_Small
- added SW1: RESET, plimsoll-Library:push_button, symbol Switch:SW_Push
- added SW2: BOOT0, plimsoll-Library:push_button, symbol Switch:SW_Push
- added U1: USBLC6-2SC6, Package_TO_SOT_SMD:SOT-23-6, symbol Power_Protection:USBLC6-2P6
- added U2: APX803L20-29SA-7, Package_TO_SOT_SMD:SOT-23, symbol onionStraws:APX803L
- added U3: STM32F072RBTx, Package_QFP:LQFP-64_10x10mm_P0.5mm, symbol MCU_ST_STM32F0:STM32F072RBTx
- added U4: AP2205-3.3, Package_TO_SOT_SMD:SOT-89-3, symbol Regulator_Linear:AP2204R-3.3
- added U5: RS3236-3.3, Package_TO_SOT_SMD:SOT-23-5, symbol Regulator_Linear:NCP163ASN350T1G
- added U6: HX717, Package_SO:SOP-16_3.9x9.9mm_P1.27mm, symbol plimsoll-symbols:HX717
Connections:
- new net: D2.1 (K), R14.1
- new net: D2.2 (A), U3.37 (PC6)
- new net: D1.1 (K), R13.1
- new net: JP1.2 (C), R10.1
- new net: R10.2, U6.6 (S0)
- new net: R11.2, U6.13 (S1)
- new net: R12.2, U6.14 (XI)
- new net: C7.1, R8.1, U6.7 (INA-)
- new net: C7.2, R7.1, U6.8 (INA+)
- new net: D1.2 (A), U3.38 (PC7)
- new net: J2.B5 (CC2), R6.1
- new net: JP2.2 (C), R11.1
- new net: J2.A5 (CC1), R5.1
- new net: J2.S1 (SHIELD), R1.2
- new net: J2.A6 (D+), J2.B6 (D+), U1.3 (I/O2)
- new net: J2.A7 (D-), J2.B7 (D-), U1.1 (I/O1)
- new net +3.3VADC: C10.1, C11.1, C12.2, C8.1, J3.4 (Pin_4), U5.5 (VOUT), U6.1 (AVDD), U6.3 (VRO/VREF), U6.4 (VFB)
- new net +3V3: C13.2, C14.2, C15.2, C16.2, C17.2, C4.1, C5.2, C9.1, J1.1 (Pin_1), JP1.1 (A), JP2.1 (A), SW1.1, SW2.1, U2.3 (Vcc), U3.1 (VBAT), U3.13 (VDDA), U3.19 (VDD), U3.32 (VDD), U3.48 (VDDIO2), U3.64 (VDD), U4.3 (VOUT), U6.16 (DVDD)
- new net BOOT0: R4.2, SW2.2, U3.60 (BOOT0)
- new net DOUT: U3.10 (PC2), U6.12 (DOUT)
- new net GND: C1.2, C10.2, C11.2, C12.1, C13.1, C14.1, C15.1, C16.1, C17.1, C2.2, C3.1, C4.2, C5.1, C6.2, C8.2, C9.2, J1.5 (Pin_5), J2.A1 (GND), J2.A12 (GND), J2.B1 (GND), J2.B12 (GND), J3.3 (Pin_3), J4.1 (Pin_1), JP1.3 (B), JP2.3 (B), R1.1, R12.1, R13.2, R14.2, R4.1, R5.2, R6.2, U1.2 (GND), U2.1 (GND), U3.12 (VSSA), U3.18 (VSS), U3.31 (VSS), U3.47 (VSS), U3.63 (VSS), U4.2 (GND), U5.2 (GND), U6.15 (DGND), U6.2 (AGND), U6.5 (AGND)
- new net PA15: J1.6 (Pin_6), U3.50 (PA15)
- new net PD_SCK: U3.9 (PC1), U6.11 (PD_SCK)
- new net SWCLK: J1.4 (Pin_4), U3.49 (PA14)
- new net SWDIO: J1.2 (Pin_2), U3.46 (PA13)
- new net Signal+: J3.1 (Pin_1), R7.2
- new net Signal-: J3.2 (Pin_2), R8.2
- new net USB_DN: U1.6 (I/O1), U3.44 (PA11)
- new net USB_DP: U1.4 (I/O2), U3.45 (PA12)
- new net VBUS: C2.1, C3.2, C6.1, J2.A4 (VBUS), J2.A9 (VBUS), J2.B4 (VBUS), J2.B9 (VBUS), J4.2 (Pin_2), U1.5 (VBUS), U4.1 (VIN), U5.1 (VIN), U5.3 (EN)
- new net nRESET: C1.1, J1.3 (Pin_3), SW1.2, U2.2 (~{RESET}), U3.7 (NRST)
- no-connect marks 0 -> 46
Other:
- note added: "Low noise, high PSSR LDO Used for analog Vdd"
- note added: "Voltage Supervisor, Hold MCU reset for 150ms after power reaches 2.9V. Prevent brownout at boot."

Commit message: r0 build details
Other:
- note added: "TODO C81720 for MCU 48 pin"
Changed lines of the file:
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@@
+		)
+	)
+	(text "TODO\n\nC81720 for MCU 48 pin"
+		(exclude_from_sim no)
+		(at 161.036 105.664 0)
+		(effects
+			(font
+				(size 1.27 1.27)
+			)
 		)
 	)
