File: mini/plimsoll.kicad_sch (KiCad schematic)
At the start: 17 parts, among them J1 Conn_02x06_Odd_Even, J3 Loadd Cell, U5 RS3236-3.3, U6 HX717

Commit message: cleanup
Other:
- note added: "Low noise, high PSSR LDO Used for analog Vdd TODO: TPS7A2033PDBVR alternative"
- note removed: "Low noise, high PSSR LDO Used for analog Vdd"
Changed lines of the file:
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@@
 		(comment 1 "CERN-OHL-S ")
 	)
-	(text "Low noise, high PSSR LDO\nUsed for analog Vdd"
+	(text "Low noise, high PSSR LDO\nUsed for analog Vdd\n\nTODO: TPS7A2033PDBVR alternative"
 		(exclude_from_sim no)
 		(at 292.1 60.198 0)
@@
 		)
 	)
+	(label "CLK"
+		(at 312.42 144.78 0)
+		(effects
+			(font
+				(size 1.27 1.27)
+			)
+			(justify left bottom)
+		)
+	)
 	(label "Signal+"
 		(at 229.87 135.89 180)
@@
 		)
 	)
+	(label "MISO"
+		(at 312.42 142.24 0)
+		(effects
+			(font
+				(size 1.27 1.27)
+			)
+			(justify left bottom)
+		)
+	)
