File: mini_ads1220/plimsoll.kicad_sch (KiCad schematic)
At the start: 17 parts, among them J1 Conn_02x06_Odd_Even, J3 Loadd Cell, U5 RS3236-3.3, U6 HX717

Commit message: ads1220 added
Parts:
- removed R10, R11, R12: 10k, Resistor_SMD:R_0603_1608Metric, symbol Device:R_Small
- removed U6: HX717, Package_SO:SOP-16_3.9x9.9mm_P1.27mm, symbol plimsoll-symbols:HX717
- added C1, C2: DNP, Capacitor_SMD:C_0603_1608Metric, symbol Device:C
- added JP2: ~{CS}, Jumper:SolderJumper-3_P1.3mm_Bridged12_RoundedPad1.0x1.5mm_NumberLabels, symbol Jumper:SolderJumper_3_Bridged12
- added U1: ADS1220xPW, Package_SO:TSSOP-16_4.4x5mm_P0.65mm, symbol Analog_ADC:ADS1220xPW
Connections:
- net +3.3VADC: now also J3.1 (Pin_1), U1.12 (AVDD), U1.9 (REFP0); no longer J3.4 (Pin_4)
- net +3V3: now also U1.13 (DVDD)
- net B3: now also U1.1 (SCLK)
- net B4: now also U1.15 (DOUT/~{DRDY})
- net B5: now also U1.16 (DIN)
- net B6: now also JP2.1 (A)
- net C13: now also U1.14 (~{DRDY})
- net GND: now also J3.2 (Pin_2), C1.1, C2.1, JP2.3 (B), U1.3 (CLK), U1.4 (DGND), U1.5 (AVSS), U1.8 (REFN0); no longer J3.3 (Pin_3)
- net Signal+: now also J3.4 (Pin_4); no longer J3.1 (Pin_1)
- net Signal-: now also J3.3 (Pin_3); no longer J3.2 (Pin_2)
- net at C7.1, R8.1: now also C1.2, U1.10 (AIN1)
- net at C7.2, R7.1: now also C2.2, U1.11 (AIN0/REFP1)
- new net: JP2.2 (C), U1.2 (~{CS})
- no-connect marks 2 -> 3
Other:
- moved on the sheet: C7, C8, C9, J3, R7, R8
