File: underbed/plimsoll.kicad_pcb (KiCad board)
At the start: 4 copper layers, 42 x 50 mm, 47 parts, among them J1 Conn_02x06_Odd_Even, U1 ADS131M04xPW, U2 RS3236-3.3, Y1 SiT8008xx-7x-xxE

Commit message: Add JLCPCB production files for three PCB projects
Other:
- board text added: "4CH Underbed Load Cell Module https://github.com/mulcmu/plimsoll"
- board text removed: "https://github.com/mulcmu/plimsoll"
Changed lines of the file:
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@@
 		(sheetname "/")
 		(sheetfile "plimsoll.kicad_sch")
-		(attr smd exclude_from_bom dnp)
+		(attr smd exclude_from_pos_files exclude_from_bom dnp)
 		(fp_line
 			(start -0.14058 0.51)
@@
 		(sheetname "/")
 		(sheetfile "plimsoll.kicad_sch")
-		(attr through_hole)
+		(attr through_hole exclude_from_pos_files exclude_from_bom)
 		(fp_line
 			(start 1.33 1.27)
@@
 		(sheetname "/")
 		(sheetfile "plimsoll.kicad_sch")
-		(attr smd exclude_from_bom dnp)
+		(attr smd exclude_from_pos_files exclude_from_bom dnp)
 		(fp_line
 			(start -0.14058 0.51)
@@
 		(sheetname "/")
 		(sheetfile "plimsoll.kicad_sch")
-		(attr through_hole exclude_from_bom)
+		(attr through_hole exclude_from_pos_files exclude_from_bom)
 		(fp_line
 			(start -1.6 -2.75)
@@
 		(sheetname "/")
 		(sheetfile "plimsoll.kicad_sch")
-		(attr smd exclude_from_bom dnp)
+		(attr smd exclude_from_pos_files exclude_from_bom dnp)
 		(fp_line
 			(start -0.14058 -0.51)
@@
 		(sheetname "/")
 		(sheetfile "plimsoll.kicad_sch")
-		(attr smd exclude_from_bom dnp)
+		(attr smd exclude_from_pos_files exclude_from_bom dnp)
 		(fp_line
 			(start -0.14058 -0.51)
@@
 		(sheetname "/")
 		(sheetfile "plimsoll.kicad_sch")
-		(attr through_hole exclude_from_bom)
+		(attr through_hole exclude_from_pos_files exclude_from_bom)
 		(fp_line
 			(start 10.06 3.51)
@@
 		(sheetname "/")
 		(sheetfile "plimsoll.kicad_sch")
-		(attr smd exclude_from_bom dnp)
+		(attr smd exclude_from_pos_files exclude_from_bom dnp)
 		(fp_line
 			(start -0.14058 -0.51)
@@
 		(sheetname "/")
 		(sheetfile "plimsoll.kicad_sch")
-		(attr through_hole exclude_from_bom)
+		(attr through_hole exclude_from_pos_files exclude_from_bom)
 		(fp_line
 			(start -2.56 3.51)
@@
 		(sheetname "/")
 		(sheetfile "plimsoll.kicad_sch")
-		(attr smd exclude_from_bom dnp)
+		(attr smd exclude_from_pos_files exclude_from_bom dnp)
 		(fp_line
 			(start -0.14058 -0.51)
@@
 		(sheetname "/")
 		(sheetfile "plimsoll.kicad_sch")
-		(attr smd exclude_from_bom dnp)
+		(attr smd exclude_from_pos_files exclude_from_bom dnp)
 		(fp_line
 			(start -0.14058 -0.51)
@@
 		(sheetname "/")
 		(sheetfile "plimsoll.kicad_sch")
-		(attr smd exclude_from_bom dnp)
+		(attr smd exclude_from_pos_files exclude_from_bom dnp)
 		(fp_line
 			(start -0.14058 -0.51)
@@
 		(sheetname "/")
 		(sheetfile "plimsoll.kicad_sch")
-		(attr through_hole exclude_from_bom)
+		(attr through_hole exclude_from_pos_files exclude_from_bom)
 		(fp_line
 			(start -2.85 -2.75)
@@
 		)
 	)
-	(gr_text "https://github.com/mulcmu/plimsoll"
-		(at 121.5 109 90)
+	(gr_text "4CH Underbed Load Cell Module\nhttps://github.com/mulcmu/plimsoll"
+		(at 116.75 123.75 90)
 		(layer "B.SilkS")
 		(effects
@@
 				(thickness 0.15)
 			)
-			(justify left bottom mirror)
+			(justify bottom mirror)
 		)
 	)
